Commit message: created another test yaml for odrive can node to test motor on node 1. i also finalized the vehicle dynamics. finally i updated the laun_sim file to automatically launch the controller spawners and remap the twistkeyboard topic publish

File: description/inertial_macros.xacro (robot description, xacro)
@@ -7,10 +7,7 @@
             <xacro:insert_block name="origin"/>
             <mass value="${mass}" />
-            <inertia ixx="2.01673334059732"
-        ixy="1.20967138671942E-08"
-        ixz="-0.0349149976927564"
-        iyy="1.89100103005672"
-        iyz="1.82499927047358E-06"
-        izz="3.72874010035965" />
+            <inertia ixx="${(2/5) * mass * (radius*radius)}" ixy="0.0" ixz="0.0"
+                    iyy="${(2/5) * mass * (radius*radius)}" iyz="0.0"
+                    izz="${(2/5) * mass * (radius*radius)}" />
         </inertial>
     </xacro:macro>
@@ -19,7 +16,11 @@
             <xacro:insert_block name="origin"/>
             <mass value="${mass}" />
-            <inertia ixx="${(1/12) * mass * (y*y+z*z)}" ixy="0.0" ixz="0.0"
-                    iyy="${(1/12) * mass * (x*x+z*z)}" iyz="0.0"
-                    izz="${(1/12) * mass * (x*x+y*y)}" />
+            <inertia
+             ixx="0.14128"
+             ixy="-1.02E-07"
+             ixz="-0.0013572"
+             iyy="0.14302"
+             iyz="6.92E-08"
+             izz="0.27183"  />
         </inertial>
     </xacro:macro>
@@ -28,7 +29,11 @@
             <xacro:insert_block name="origin"/>
             <mass value="${mass}" />
-            <inertia ixx="${(1/12) * mass * (3*radius*radius + length*length)}" ixy="0.0" ixz="0.0"
-                    iyy="${(1/12) * mass * (3*radius*radius + length*length)}" iyz="0.0"
-                    izz="${(1/2) * mass * (radius*radius)}" />
+            <inertia
+             ixx="0.00120506"
+             ixy="6.67E-09"
+             ixz="-2.51E-10"
+             iyy="0.001205041"
+             iyz="-7.22E-10"
+             izz="0.002290365" />
         </inertial>
     </xacro:macro>

File: description/robot_core.xacro (robot description, xacro)
@@ -36,6 +36,6 @@
             </geometry>
         </collision>
-        <xacro:inertial_box mass="67.4001728547215" x="0.46" y="0.46" z="0.3">
-            <origin xyz="-0.04 0.0 0.115" rpy="0.0 0.0 0.0"/>
+        <xacro:inertial_box mass="10.319" x="0.46" y="0.46" z="0.3">
+            <origin xyz="-0.14743 -0.00064615 0.027414" rpy="0.0 0.0 0.0"/>
         </xacro:inertial_box>
     </link>
@@ -60,8 +60,8 @@
         <origin xyz="0.0 0.0 0.0" rpy="0.0 0.0 0.0"/>
         <geometry>
-            <cylinder radius="0.083" length="0.04"/>
+            <sphere radius="0.083"/>
         </geometry>
     </collision>
-    <xacro:inertial_cylinder mass="0.522473609523098" length="0.4" radius="0.083">
+    <xacro:inertial_cylinder mass="0.454027315" length="0.4" radius="0.083">
     <origin xyz="0.0 0.0 0.0" rpy="0.0 0.0 0.0"/>
     </xacro:inertial_cylinder>
@@ -86,8 +86,8 @@
     <collision>
         <geometry>
-            <cylinder radius="0.083" length="0.04"/>
+            <sphere radius="0.083"/>
         </geometry>
     </collision>
-    <xacro:inertial_cylinder mass="0.522473609523098" length="0.4" radius="0.083">
+    <xacro:inertial_cylinder mass="0.454027315" length="0.4" radius="0.083">
     <origin xyz="0.0 0.0 0.0" rpy="0.0 0.0 0.0"/>
     </xacro:inertial_cylinder>

File: urdf/urdf/Shared_Assembly_Robot_URDF.urdf (robot description, URDF)
Before this commit: robot Shared_Assembly_Robot_URDF, 8 links, 7 joints
Links:
- link base_link: mass 67.4001728547215 -> 10.319
- link left_wheel: mass 0.522473586119869 -> 0.454027333
- link right_wheel: mass 0.522473609523098 -> 0.454027315
