Commit message: Fixed URDF file and created a configuration file for Rviz

File: description/robot_core.xacro (robot description, xacro)
@@ -36,5 +36,4 @@
         <parent link="base_link"/>
         <child link="left_wheel"/>
-        <axis xyz="0 0 0"/>
         <origin xyz="0 0.175 0" rpy="-${pi/2} 0 0"/>
         <axis xyz="0.0 0.0 1.0"/>
@@ -61,5 +60,4 @@
         <parent link="base_link"/>
         <child link="right_wheel"/>
-        <axis xyz="0 0 0"/>
         <origin xyz="0 -0.175 0" rpy="${pi/2} 0 0"/>
         <axis xyz="0.0 0.0 -1.0"/>

Commit message: modified urdf to push wheels to from of robot

File: description/robot_core.xacro (robot description, xacro)
@@ -16,5 +16,5 @@
     <link name="chassis">
         <visual>
-            <origin xyz="0.15 0.0 0.075" rpy="0.0 0.0 0.0"/>
+            <origin xyz="0.01 0.0 0.075" rpy="0.0 0.0 0.0"/>
             <geometry>
                 <box size="0.3 0.3 0.15"/>
@@ -23,5 +23,5 @@
         </visual>
         <collision>
-            <origin xyz="0.15 0.0 0.075" rpy="0.0 0.0 0.0"/>
+            <origin xyz="0.01 0.0 0.075" rpy="0.0 0.0 0.0"/>
             <geometry>
                 <box size="0.3 0.3 0.15"/>
@@ -29,5 +29,5 @@
         </collision>
         <xacro:inertial_box mass="0.5" x="0.3" y="0.3" z="0.1">
-            <origin xyz="0.15 0.0 0.075" rpy="0.0 0.0 0.0"/>
+            <origin xyz="0.01 0.0 0.075" rpy="0.0 0.0 0.0"/>
         </xacro:inertial_box>
     </link>
@@ -92,5 +92,5 @@
         <parent link="chassis"/>
         <child link="caster_wheel"/>
-        <origin xyz="0.24 0.0 0.0" rpy="0.0 0.0 0.0"/>
+        <origin xyz="-.085 0.0 0.0" rpy="0.0 0.0 0.0"/>
     </joint>
     <link name="caster_wheel">
@@ -99,5 +99,5 @@
                 <sphere radius="0.05"/>
             </geometry>
-            <material name="black" />
+            <material name="orange" />
         </visual>
         <collision>

Commit message: set up slam

File: description/robot_core.xacro (robot description, xacro)
@@ -7,4 +7,12 @@
     <!-- BASE LINK  -->
     <link name="base_link">
+    </link>
+    <!-- BASE_FOOTPRINT LINK -->
+    <joint name="base_footprint_joint" type="fixed">
+        <parent link="base_link"/>
+        <child link="base_footprint"/>
+        <origin xyz="0 0 0" rpy="0 0 0"/>
+    </joint>
+    <link name="base_footprint">
     </link>
     <!-- CHASSIS LINK -->

Commit message: can now drive the physical robot via ps4 controller

File: description/robot_core.xacro (robot description, xacro)
@@ -47,5 +47,5 @@
         <parent link="base_link"/>
         <child link="left_wheel"/>
-        <origin xyz="0 0.25 0" rpy="-${pi/2} 0 0"/>
+        <origin xyz="0 0.25 0" rpy="${pi/2} 0 0"/>
         <axis xyz="0.0 0.0 1.0"/>
     </joint>
